File: schemi/Driver_motore/Driver_motore_v2/Driver_motore_v2.kicad_sch (KiCad schematic)
At the start: 44 parts, among them J1 PICKIT, J2 Motore, J3 Power, J4 Conn, J5 controllo_motore, J6 controllo_encoder, J7 controllo_alimentazione, M1 Motor_DC, U1 L298N, U2 PIC16F88-IP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

Commit message: update main board
Other:
- moved on the sheet: H1, H2, H3, H4
Changed lines of the file:
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@@
 	)
 	(rectangle
-		(start 142.24 116.84)
-		(end 175.26 146.05)
+		(start 156.21 133.35)
+		(end 189.23 162.56)
 		(stroke
 			(width 0)
@@
 	(text "FORI DI MONTAGGIO"
 		(exclude_from_sim no)
-		(at 160.02 115.57 0)
+		(at 173.99 132.08 0)
 		(effects
 			(font
@@
 	)
 	(junction
-		(at 146.05 130.81)
+		(at 160.02 147.32)
 		(diameter 0)
 		(color 0 0 0 0)
@@
 	)
 	(junction
-		(at 146.05 135.89)
+		(at 160.02 152.4)
 		(diameter 0)
 		(color 0 0 0 0)
@@
 	)
 	(junction
-		(at 146.05 125.73)
+		(at 160.02 142.24)
 		(diameter 0)
 		(color 0 0 0 0)
@@
 	(wire
 		(pts
-			(xy 146.05 125.73) (xy 146.05 130.81)
+			(xy 160.02 142.24) (xy 160.02 147.32)
 		)
 		(stroke
@@
 	(wire
 		(pts
-			(xy 146.05 120.65) (xy 147.32 120.65)
+			(xy 160.02 137.16) (xy 161.29 137.16)
 		)
 		(stroke
@@
 	(wire
 		(pts
-			(xy 146.05 135.89) (xy 146.05 138.43)
+			(xy 160.02 152.4) (xy 160.02 154.94)
 		)
 		(stroke
@@
 	(wire
 		(pts
-			(xy 147.32 125.73) (xy 146.05 125.73)
+			(xy 161.29 142.24) (xy 160.02 142.24)
 		)
 		(stroke
@@
 	(wire
 		(pts
-			(xy 146.05 120.65) (xy 146.05 125.73)
+			(xy 160.02 137.16) (xy 160.02 142.24)
 		)
 		(stroke
@@
 	(wire
 		(pts
-			(xy 146.05 130.81) (xy 146.05 135.89)
+			(xy 160.02 147.32) (xy 160.02 152.4)
 		)
 		(stroke
@@
 	(wire
 		(pts
-			(xy 147.32 130.81) (xy 146.05 130.81)
+			(xy 161.29 147.32) (xy 160.02 147.32)
 		)
 		(stroke
@@
 	(wire
 		(pts
-			(xy 146.05 135.89) (xy 147.32 135.89)
+			(xy 160.02 152.4) (xy 161.29 152.4)
 		)
 		(stroke
@@
 	(symbol
 		(lib_id "Mechanical:MountingHole_Pad")
-		(at 149.86 125.73 270)
+		(at 163.83 142.24 270)
 		(unit 1)
 		(body_style 1)
@@
 		(fields_autoplaced yes)
 		(property "Reference" "H2"
-			(at 153.67 124.4599 90)
+			(at 167.64 140.9699 90)
 			(show_name no)
 			(do_not_autoplace no)
@@
 		)
 		(property "Value" "MountingHole_Pad"
-			(at 153.67 126.9999 90)
+			(at 167.64 143.5099 90)
 			(show_name no)
 			(do_not_autoplace no)
@@
 		)
 		(property "Footprint" "MountingHole:MountingHole_2.5mm_Pad"
-			(at 149.86 125.73 0)
+			(at 163.83 142.24 0)
 			(hide yes)
 			(show_name no)
@@
 		)
 		(property "Datasheet" ""
-			(at 149.86 125.73 0)
+			(at 163.83 142.24 0)
 			(hide yes)
 			(show_name no)
@@
 		)
 		(property "Description" "Mounting Hole with connection"
-			(at 149.86 125.73 0)
+			(at 163.83 142.24 0)
 			(hide yes)
 			(show_name no)
@@
 	(symbol
 		(lib_id "power:GND")
-		(at 146.05 138.43 0)
+		(at 160.02 154.94 0)
 		(unit 1)
 		(body_style 1)
@@
 		(fields_autoplaced yes)
 		(property "Reference" "#PWR025"
-			(at 146.05 144.78 0)
+			(at 160.02 161.29 0)
 			(hide yes)
 			(show_name no)
@@
 		)
 		(property "Value" "GND"
-			(at 146.05 143.51 0)
+			(at 160.02 160.02 0)
 			(show_name no)
 			(do_not_autoplace no)
@@
 		)
 		(property "Footprint" ""
-			(at 146.05 138.43 0)
+			(at 160.02 154.94 0)
 			(hide yes)
 			(show_name no)
@@
 		)
 		(property "Datasheet" ""
-			(at 146.05 138.43 0)
+			(at 160.02 154.94 0)
 			(hide yes)
 			(show_name no)
@@
 		)
 		(property "Description" "Power symbol creates a global label with name \"GND\" , ground"
-			(at 146.05 138.43 0)
+			(at 160.02 154.94 0)
 			(hide yes)
 			(show_name no)
@@
 	(symbol
 		(lib_id "Mechanical:MountingHole_Pad")
-		(at 149.86 135.89 270)
+		(at 163.83 152.4 270)
 		(unit 1)
 		(body_style 1)
@@
 		(fields_autoplaced yes)
 		(property "Reference" "H4"
-			(at 153.67 134.6199 90)
+			(at 167.64 151.1299 90)
 			(show_name no)
 			(do_not_autoplace no)
@@
 		)
 		(property "Value" "MountingHole_Pad"
-			(at 153.67 137.1599 90)
+			(at 167.64 153.6699 90)
 			(show_name no)
 			(do_not_autoplace no)
@@
 		)
 		(property "Footprint" "MountingHole:MountingHole_2.5mm_Pad"
-			(at 149.86 135.89 0)
+			(at 163.83 152.4 0)
 			(hide yes)
 			(show_name no)
@@
 		)
 		(property "Datasheet" ""
-			(at 149.86 135.89 0)
+			(at 163.83 152.4 0)
 			(hide yes)
 			(show_name no)
@@
 		)
 		(property "Description" "Mounting Hole with connection"
-			(at 149.86 135.89 0)
+			(at 163.83 152.4 0)
 			(hide yes)
 			(show_name no)
@@
 	(symbol
 		(lib_id "Mechanical:MountingHole_Pad")
-		(at 149.86 120.65 270)
+		(at 163.83 137.16 270)
 		(unit 1)
 		(body_style 1)
@@
 		(fields_autoplaced yes)
 		(property "Reference" "H1"
-			(at 153.67 119.3799 90)
+			(at 167.64 135.8899 90)
 			(show_name no)
 			(do_not_autoplace no)
@@
 		)
 		(property "Value" "MountingHole_Pad"
-			(at 153.67 121.9199 90)
+			(at 167.64 138.4299 90)
 			(show_name no)
 			(do_not_autoplace no)
@@
 		)
 		(property "Footprint" "MountingHole:MountingHole_2.5mm_Pad"
-			(at 149.86 120.65 0)
+			(at 163.83 137.16 0)
 			(hide yes)
 			(show_name no)
@@
 		)
 		(property "Datasheet" ""
-			(at 149.86 120.65 0)
+			(at 163.83 137.16 0)
 			(hide yes)
 			(show_name no)
@@
 		)
 		(property "Description" "Mounting Hole with connection"
-			(at 149.86 120.65 0)
+			(at 163.83 137.16 0)
 			(hide yes)
 			(show_name no)
@@
 	(symbol
 		(lib_id "Mechanical:MountingHole_Pad")
-		(at 149.86 130.81 270)
+		(at 163.83 147.32 270)
 		(unit 1)
 		(body_style 1)
@@
 		(fields_autoplaced yes)
 		(property "Reference" "H3"
-			(at 153.67 129.5399 90)
+			(at 167.64 146.0499 90)
 			(show_name no)
 			(do_not_autoplace no)
@@
 		)
 		(property "Value" "MountingHole_Pad"
-			(at 153.67 132.0799 90)
+			(at 167.64 148.5899 90)
 			(show_name no)
 			(do_not_autoplace no)
@@
 		)
 		(property "Footprint" "MountingHole:MountingHole_2.5mm_Pad"
-			(at 149.86 130.81 0)
+			(at 163.83 147.32 0)
 			(hide yes)
 			(show_name no)
@@
 		)
 		(property "Datasheet" ""
-			(at 149.86 130.81 0)
+			(at 163.83 147.32 0)
 			(hide yes)
 			(show_name no)
@@
 		)
 		(property "Description" "Mounting Hole with connection"
-			(at 149.86 130.81 0)
+			(at 163.83 147.32 0)
 			(hide yes)
 			(show_name no)
