File: schemi/Driver_motore/Driver_motore_v2/Driver_motore_v2.kicad_sch (KiCad schematic)
At the start: 44 parts, among them J1 PICKIT, J2 Motore, J3 Power, J4 Conn, J5 controllo_motore, J6 controllo_encoder, J7 controllo_alimentazione, M1 Motor_DC, U1 L298N, U2 PIC16F88-IP, U3 LM7805_TO220

Commit message: update generale
Parts:
- R1: value R -> 10k
- R2: value R -> 1k
Changed lines of the file:
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@@
 			)
 		)
-		(property "Value" "R"
+		(property "Value" "1k"
 			(at 116.84 170.1799 0)
 			(show_name no)
@@
 			)
 		)
-		(property "Value" "R"
+		(property "Value" "10k"
 			(at 59.69 170.1799 0)
 			(show_name no)
