File: schemi/main_board/main_board.kicad_sch (KiCad schematic)
At the start: 73 parts, among them J1 PICKIT, J10 sensore_temp, J2 FC1, J3 FC2, J4 Conn_Relè, J5 MOTORE, J6 Power_barrel, J7 sensore_temp, J8 Power, J9 controllo_alimentazione, K1 Ventilazione, K2 finestre, K3 acqua, Q1 2N2222A, Q2 2N2222A, Q3 2N2222A, Q4 2N2222A, Q5 2N2222A, SW1 START, SW2 STOP, SW3 MODO, U1 PIC16F887-IP, U2 LM35-LP, U4 LM7805_TO220, U5 SM420561N, U6 SM420561N

Commit message: update generale
Parts:
- added C1: 100nF, symbol Device:C
- added R10: 1k, symbol Device:R
- R11, R23, R31, R32: value R -> 10k
- R17, R19, R30: value 1K -> 1k
- R8, R9: value R -> 1k
Connections:
- net GND: now also C1.2
- net at J10.2 (Pin_2): now also R10.2; no longer U2.2 (V_{OUT})
- new net: C1.1, R10.1, U2.2 (V_{OUT})
Other:
- moved on the sheet: J10, U2
